File: kicad10-project-template.kicad_sch (KiCad schematic)
At the start: 0 parts

Commit message: Revert "test"
This reverts commit ebfcfdce2563dfeda8234330652bd01ca862520f.
Other:
- company: DonanimKafa -> (none)
Changed lines of the file:
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@@
 	(generator_version "10.0")
 	(paper "A4")
-	(title_block
-		(company "DonanimKafa")
-		(comment 1 "PHASE: draft")
-	)
 	(sheet_instances
 		(path "/"

Commit message: test
Other:
- company: (none) -> DonanimKafa
Changed lines of the file:
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@@
 	(generator_version "10.0")
 	(paper "A4")
+	(title_block
+		(company "DonanimKafa")
+		(comment 1 "PHASE: draft")
+	)
 	(sheet_instances
 		(path "/"
