File: hardware/kicad10-project-template.kicad_sch (KiCad schematic)
At the start: 0 parts

Commit message: ci(workflow): release PHASE koşuluna bağlandı, git güvenli dizin ve tam geçmiş eklendi
Release işi artık yalnızca v* etiketi ve şematikteki PHASE değeri release ise çalışır; faz değeri build işinin çıktısıyla aktarılır. Konteynerde git dubious ownership hatasını önlemek için safe.directory ayarı ve etiketlerin bulunması için fetch-depth 0 eklendi. action-gh-release v2 sürümüne yükseltildi, timeout ve concurrency eklendi.
Other:
- company: DonanimKafa -> (none)
Changed lines of the file:
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@@
 	(generator_version "10.0")
 	(paper "A4")
-	(title_block
-		(company "DonanimKafa")
-		(comment 1 "PHASE: draft")
-	)
-	(symbol
-		(lib_id "PCM_SparkFun-PowerSymbol:0.9V")
-		(at 130.81 63.5 0)
-		(unit 1)
-		(body_style 1)
-		(exclude_from_sim no)
-		(in_bom yes)
-		(on_board yes)
-		(in_pos_files yes)
-		(dnp no)
-		(fields_autoplaced yes)
-		(property "Reference" "#PWR01"
-			(at 130.81 67.31 0)
-			(hide yes)
-			(show_name no)
-			(do_not_autoplace no)
-			(effects
-				(font
-					(size 1.27 1.27)
-				)
-			)
-		)
-		(property "Value" "0.9V"
-			(at 130.81 59.69 0)
-			(show_name no)
-			(do_not_autoplace yes)
-			(effects
-				(font
-					(size 1.27 1.27)
-				)
-			)
-		)
-		(property "Footprint" ""
-			(at 130.81 63.5 0)
-			(hide yes)
-			(show_name no)
-			(do_not_autoplace no)
-			(effects
-				(font
-					(size 1.27 1.27)
-				)
-			)
-		)
-		(property "Datasheet" ""
-			(at 130.81 63.5 0)
-			(hide yes)
-			(show_name no)
-			(do_not_autoplace no)
-			(effects
-				(font
-					(size 1.27 1.27)
-				)
-			)
-		)
-		(property "Description" "Power symbol creates a global label with name \"0.9V\""
-			(at 130.81 69.85 0)
-			(hide yes)
-			(show_name no)
-			(do_not_autoplace no)
-			(effects
-				(font
-					(size 1.27 1.27)
-				)
-			)
-		)
-		(pin "1"
-		)
-		(instances
-			(project "kicad10-project-template"
-				(path "/7e15e6e1-e0da-4828-9eff-01b53389ad0b"
-					(reference "#PWR01")
-					(unit 1)
-				)
-			)
-		)
-	)
 	(sheet_instances
 		(path "/"

Commit message: fix(title-block): betik KiCad dosyalarını hardware klasöründe arar
update_title_block.py tek başına çalıştırıldığında .kicad_sch ve .kicad_pcb dosyalarını artık varsayılan olarak hardware/ klasöründe arar. Yeni --hardware-dir argümanı eklendi; klasör yoksa proje köküne geri düşülür. build_docs.py üzerinden kullanımda davranış değişmedi.
Other:
- company: (none) -> Donanimkafa
Changed lines of the file:
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@@
 	)
 	(embedded_fonts no)
+(title_block
+  (rev "v1.0.0")
+  (date "2026-10-21")
+  (company "Donanimkafa")
 )
+)

Commit message: docs(Sheet) Sayfa hiyerarşileri ve sayfa yapıları düzenlendi.
Other:
- added sheet Block Diagram (Block Diagram.kicad_sch)
- added sheet Power - Sequencing (Power - Sequencing.kicad_sch)
- added sheet Project Architecture (Project Architecture.kicad_sch)
- added sheet Revision History (Revision History.kicad_sch)
- note added: "${BOARD_NAME}"
- note added: "${ISSUE_DATE}"
- note added: "${PROJECT_DESCRIPTION}"
- note added: "${SHEET_NAME_10}"
- note added: "${SHEET_NAME_1}"
- note added: "${SHEET_NAME_2}"
- note added: "${SHEET_NAME_3}"
- note added: "${SHEET_NAME_4}"
- note added: "${SHEET_NAME_5}"
- note added: "${SHEET_NAME_6}"
- note added: "${SHEET_NAME_7}"
- note added: "${SHEET_NAME_8}"
- note added: "${SHEET_NAME_9}"
- note added: "..................................."
- note added: "1"
- note added: "10"
- note added: "11"
- note added: "12"
- note added: "13"
- note added: "14"
- note added: "15"
- note added: "16"
- note added: "17"
- note added: "18"
- note added: "19"
- note added: "2"
- note added: "20"
- note added: "21"
- note added: "22"
- note added: "23"
- note added: "24"
- note added: "25"
- note added: "26"
- note added: "27"
- note added: "28"
- note added: "29"
- note added: "3"
- note added: "30"
- note added: "31"
- note added: "32"
- note added: "33"
- note added: "34"
- note added: "35"
- note added: "36"
- note added: "37"
- note added: "38"
- note added: "39"
- note added: "4"
- note added: "40"
- note added: "5"
- note added: "6"
- note added: "7"
- note added: "8"
- note added: "9"
- note added: "ALT GÖRÜNÜŞ"
- note added: "BÖLÜM"
- note added: "BİLGİ"
- note added: "DRAFT / Şematik geliştirme aşamasında. PRELIMINARY / Ön inceleme; bulgular olabilir. CHECKED / ERC ve DRC kontrolleri zorunlu. RELEASE / Onaylı üretim sürümü."
- note added: "DİKKAT"
- note added: "FAZ: ${PHASE} | PROJE: ${PROJECT_CODE}"
- note added: "Genel tasarım açıklamaları."
- note added: "Güç ve güvenlik kontrolleri."
- note added: "KRİTİK"
- note added: "LAYOUT"
- note added: "PCB görseli buraya eklenir"
- note added: "PROJE NOTLARI"
- note added: "Parça seçimi ve montaj notları."
- note added: "REV: ${REVISION}"
- note added: "SAYFA"
- note added: "TASARIM NOTLARI"
- note added: "Yerleşim ve iz yönlendirme."
- note added: "ÜST GÖRÜNÜŞ"
- note added: "İçindekiler elle güncellenir. PCB görselleri otomatik oluşturulmaz. Üretim için etiketli Release dosyalarını kullanın."
- note added: "ŞEMATİK İÇİNDEKİLER"
- title: (none) -> ${BOARD_NAME}
