File: hardware/Block Diagram.kicad_sch (KiCad schematic)
At the start: 0 parts

Commit message: docs(readme): güncel proje yapısını ve kullanımını belgele
README'yi hiyerarşik şematikler, proje değişkenleri, BOM ve net ayarlarıyla güncelle. Üretim ve CI davranışını açıklığa kavuştur.
Other:
- note added: "+??V"
- note added: "+A3V3"
